Commit message: Create new urdf xacro file in amr_lan_3.

File: src/amr_lan_2_mesh/description/robot.urdf.xacro (robot description, xacro)
@@ -4,5 +4,5 @@
     <!-- <link name="base_footprint"></link> -->
     <xacro:include filename="robot_core.xacro" />
-    <xacro:include filename="gazebo_control.xacro" />
+    <!-- <xacro:include filename="gazebo_control.xacro" /> -->
     <xacro:include filename="lidar.xacro" />
     <xacro:include filename="ros2_control.xacro" />

File: src/amr_lan_2_mesh/description/ros2_control.xacro (robot description, xacro)
@@ -19,2 +19,31 @@
     </ros2_control>
 </robot>
+<!-- <?xml version="1.0"?>
+<robot xmlns:xacro="http://www.ros.org/wiki/xacro">
+    <ros2_control name="GazeboSystem" type="system">
+        <hardware>
+            <plugin>gazebo_ros2_control/GazeboSystem</plugin>
+        </hardware>
+        <joint name="left_wheel_joint">
+            <command_interface name="velocity">
+                <param name="min">-1</param>
+                <param name="max">1</param>
+            </command_interface>
+            <state_interface name="velocity"/>
+            <state_interface name="position"/>
+        </joint>
+        <joint name="right_wheel_joint">
+            <command_interface name="velocity">
+                <param name="min">-1</param>
+                <param name="max">1</param>
+            </command_interface>
+            <state_interface name="velocity"/>
+            <state_interface name="position"/>
+        </joint>
+    </ros2_control>
+    <gazebo>
+        <plugin name="gazebo_ros2_control" filename="libgazebo_ros2_control.so">
+            <parameters>$(find amr_lan_2_mesh)/config/controllers.yaml</parameters>
+        </plugin>
+    </gazebo>
+</robot> -->
