Commit message: add gazebo plguin to drive virtual robot in gazebo.

File: src/amr_lan_3/description/lidar.xacro (robot description, xacro)
@@ -15,12 +15,6 @@
             <geometry>
                 <cylinder radius="0.035" length="0.04"/>
-                <!-- <mesh filename="package://amr_lan_2_mesh/meshes/laser_frame.STL"/> -->
             </geometry>
-            <material
-                name="">
-                <color
-                rgba="0.211764705882353 0.211764705882353 0.203921568627451 1"/>
-                <!-- <color name="xanhlo"/> -->
-            </material>
+            <material name="black"/>
         </visual>
         <collision>
@@ -28,10 +22,9 @@
             <geometry>
                 <cylinder radius="0.035" length="0.04"/>
-                <!-- <mesh filename="package://amr_lan_2_mesh/meshes/laser_frame.STL"/> -->
             </geometry>
         </collision>
-        <!-- <xacro:inertial_cylinder mass="0.1" length="0.04" radius="0.035">
+        <xacro:inertial_cylinder mass="0.1" length="0.04" radius="0.035">
             <origin xyz="0 0 0" rpy="0 0 0"/>
-        </xacro:inertial_cylinder> -->
+        </xacro:inertial_cylinder>
     </link>
     <!-- <gazebo reference="laser_frame">

File: src/amr_lan_3/description/robot.urdf.xacro (robot description, xacro)
@@ -2,5 +2,5 @@
 <robot xmlns:xacro="http://www.ros.org/wiki/xacro" name="robot">
     <xacro:include filename="robot_core.xacro" />
-    <!-- <xacro:include filename="gazebo_control.xacro" /> -->
+    <xacro:include filename="gazebo_control.xacro" />
     <xacro:include filename="lidar.xacro" />
     <!-- <xacro:include filename="ros2_control.xacro" /> -->

File: src/amr_lan_3/description/robot_core.xacro (robot description, xacro)
@@ -59,7 +59,7 @@
         </xacro:inertial_box>
     </link>
-    <!-- <gazebo reference="base_link">
+    <gazebo reference="base_link">
         <material>Gazebo/Green</material>
-    </gazebo> -->
+    </gazebo>
      <!-- CHASSIS 1 LINK -->
     <joint name="chassis_1_joint" type="fixed">
@@ -86,7 +86,7 @@
         </xacro:inertial_box>
     </link>
-    <!-- <gazebo reference="base_link">
-        <material>Gazebo/Green</material>
-    </gazebo> -->
+    <gazebo reference="chassis_1_link">
+        <material>Gazebo/Orange</material>
+    </gazebo>
     <!-- LEFT WHEEL LINK -->
     <joint name="left_wheel_joint" type="continuous">
@@ -114,9 +114,9 @@
         </xacro:inertial_cylinder>
     </link>
-    <!-- <gazebo reference="left_wheel">
+    <gazebo reference="left_wheel">
         <material>Gazebo/Purple</material>
-        <mu1 value="0.4"/>
-        <mu2 value="0.4"/>
-    </gazebo> -->
+        <mu1 value="0.7"/>
+        <mu2 value="0.7"/>
+    </gazebo>
     <!-- RIGHT WHEEL LINK -->
     <joint name="right_wheel_joint" type="continuous">
@@ -144,9 +144,9 @@
         </xacro:inertial_cylinder>
     </link>
-    <!-- <gazebo reference="right_wheel">
+    <gazebo reference="right_wheel">
         <material>Gazebo/Purple</material>
-        <mu1 value="0.4"/>
-        <mu2 value="0.4"/>
-    </gazebo> -->
+        <mu1 value="0.7"/>
+        <mu2 value="0.7"/>
+    </gazebo>
     <!-- CASTER WHEEL RIGHT BEHIND LINK -->
     <joint name="caster_wheel_right_behind_joint" type="fixed">
@@ -173,11 +173,11 @@
         </xacro:inertial_sphere>
     </link>
-    <!-- <gazebo reference="caster_wheel_right_behind">
-        <material>Gazebo/Blue</material>
-        <mu1 value="0"/>
-        <mu2 value="0"/>
-        <slip1>1.0</slip1>
-        <slip2>1.0</slip2>
-    </gazebo> -->
+    <gazebo reference="caster_wheel_right_behind">
+        <material>Gazebo/Blue</material>
+        <mu1 value="0"/>
+        <mu2 value="0"/>
+        <!-- <slip1>1.0</slip1>
+        <slip2>1.0</slip2> -->
+    </gazebo>
     <!-- CASTER WHEEL LEFT BEHIND LINK -->
     <joint name="caster_wheel_left_behind_joint" type="fixed">
@@ -204,11 +204,11 @@
         </xacro:inertial_sphere>
     </link>
-    <!-- <gazebo reference="caster_wheel_left_behind">
-        <material>Gazebo/Blue</material>
-        <mu1 value="0"/>
-        <mu2 value="0"/>
-        <slip1>1.0</slip1>
-        <slip2>1.0</slip2>
-    </gazebo> -->
+    <gazebo reference="caster_wheel_left_behind">
+        <material>Gazebo/Blue</material>
+        <mu1 value="0"/>
+        <mu2 value="0"/>
+        <!-- <slip1>1.0</slip1>
+        <slip2>1.0</slip2> -->
+    </gazebo>
     <!-- CASTER WHEEL RIGHT FRONT LINK -->
     <joint name="caster_wheel_right_front_joint" type="fixed">
@@ -235,11 +235,11 @@
         </xacro:inertial_sphere>
     </link>
-    <!-- <gazebo reference="caster_wheel_right_front">
-        <material>Gazebo/Blue</material>
-        <mu1 value="0"/>
-        <mu2 value="0"/>
-        <slip1>1.0</slip1>
-        <slip2>1.0</slip2>
-    </gazebo> -->
+    <gazebo reference="caster_wheel_right_front">
+        <material>Gazebo/Blue</material>
+        <mu1 value="0"/>
+        <mu2 value="0"/>
+        <!-- <slip1>1.0</slip1>
+        <slip2>1.0</slip2> -->
+    </gazebo>
     <!-- CASTER WHEEL LEFT FRONT LINK -->
     <joint name="caster_wheel_left_front_joint" type="fixed">
@@ -266,10 +266,10 @@
         </xacro:inertial_sphere>
     </link>
-    <!-- <gazebo reference="caster_wheel_left_front">
-        <material>Gazebo/Blue</material>
-        <mu1 value="0"/>
-        <mu2 value="0"/>
-        <slip1>1.0</slip1>
-        <slip2>1.0</slip2>
-    </gazebo> -->
+    <gazebo reference="caster_wheel_left_front">
+        <material>Gazebo/Blue</material>
+        <mu1 value="0"/>
+        <mu2 value="0"/>
+        <!-- <slip1>1.0</slip1>
+        <slip2>1.0</slip2> -->
+    </gazebo>
 </robot>

Commit message: Done vid 1 ROS2_control
    Adding file controllers.yaml and ros2_control.xacro for simulate driving robot

Modifier 2 file:

    robot.urdf.xacro (include ros2_control.xacro and comment gazebo_control.xacro)

launch_sim.launch.py (Adding 2 ros2_control Node and spawner it)

ROBOT HAS DRIFF WHEN SIMULATE, STILL HAVEN'T FIX

File: src/amr_lan_3/description/lidar.xacro (robot description, xacro)
@@ -28,6 +28,6 @@
         </xacro:inertial_cylinder>
     </link>
-    <!-- <gazebo reference="laser_frame">
-        <material>Gazebo/Red</material>
+    <gazebo reference="laser_frame">
+        <!-- <material>Gazebo/Red</material> -->
         <material>Gazebo/Black</material>
         <sensor name="laser" type="ray">
@@ -49,9 +49,9 @@
                     <resolution>0.01</resolution>
                 </range>
-                <noise>
+                <!-- <noise>
                     <type>gaussian</type>
                     <mean>0.0</mean>
                     <stddev>0.01</stddev> Small noise for realism
-                </noise>
+                </noise> -->
             </ray>
             <plugin name="laser_controller" filename="libgazebo_ros_ray_sensor.so">
@@ -63,4 +63,4 @@
             </plugin>
         </sensor>
-    </gazebo> -->
+    </gazebo>
 </robot>

File: src/amr_lan_3/description/robot.urdf.xacro (robot description, xacro)
@@ -2,6 +2,6 @@
 <robot xmlns:xacro="http://www.ros.org/wiki/xacro" name="robot">
     <xacro:include filename="robot_core.xacro" />
-    <xacro:include filename="gazebo_control.xacro" />
+    <xacro:include filename="ros2_control.xacro" />
+    <!-- <xacro:include filename="gazebo_control.xacro" /> -->
     <xacro:include filename="lidar.xacro" />
-    <!-- <xacro:include filename="ros2_control.xacro" /> -->
 </robot>

File: src/amr_lan_3/description/robot_core.xacro (robot description, xacro)
@@ -72,5 +72,5 @@
             <origin xyz="0 0 0"/>
             <geometry>
-                <box size="1.0 0.5 0.06"/>
+                <box size="1.04 0.51 0.06"/>
             </geometry>
             <material name="vibrantorange"/>
@@ -79,5 +79,5 @@
             <origin xyz="0 0 0"/>
             <geometry>
-                <box size="1.0 0.5 0.06"/>
+                <box size="1.04 0.51 0.06"/>
             </geometry>
         </collision>
