Commit message: Laptop_driver_ros2_control
    Fix read_function, hall_sensor, in hinson package

Haven't run sim robot in gazebo again

File: src/amr_lan_3/description/robot_core.xacro (robot description, xacro)
@@ -107,5 +107,6 @@
             <origin xyz="0 0 0"/>
             <geometry>
-                <cylinder radius="0.09" length="0.04"/>
+                <!-- <cylinder radius="0.09" length="0.04"/> -->
+            <sphere radius="0.09"/>
             </geometry>
         </collision>
@@ -116,6 +117,6 @@
     <gazebo reference="left_wheel">
         <material>Gazebo/Purple</material>
-        <mu1 value="0.7"/>
-        <mu2 value="0.7"/>
+        <mu1 value="10.0"/>
+        <mu2 value="10.0"/>
     </gazebo>
     <!-- RIGHT WHEEL LINK -->
@@ -137,5 +138,6 @@
             <origin xyz="0 0 0"/>
             <geometry>
-                <cylinder radius="0.09" length="0.04"/>
+                <!-- <cylinder radius="0.09" length="0.04"/> -->
+                <sphere radius="0.09"/>
             </geometry>
         </collision>
@@ -146,6 +148,6 @@
     <gazebo reference="right_wheel">
         <material>Gazebo/Purple</material>
-        <mu1 value="0.7"/>
-        <mu2 value="0.7"/>
+        <mu1 value="10.0"/>
+        <mu2 value="10.0"/>
     </gazebo>
     <!-- CASTER WHEEL RIGHT BEHIND LINK -->

File: src/amr_lan_3/description/ros2_control.xacro (robot description, xacro)
@@ -1,2 +1,23 @@
+<?xml version="1.0"?>
+<robot xmlns:xacro="http://www.ros.org/wiki/xacro">
+    <ros2_control name="RealRobot" type="system">
+        <hardware>
+            <plugin>hinson_hardware/HinsonSystemHardware</plugin>
+            <param name="port">/dev/ttyUSB0</param>
+            <param name="baudrate">115200</param>
+        </hardware>
+        <joint name="left_wheel_joint">
+            <command_interface name="velocity"/>
+            <state_interface name="position"/>
+            <state_interface name="velocity"/>
+        </joint>
+        <joint name="right_wheel_joint">
+            <command_interface name="velocity"/>
+            <state_interface name="position"/>
+            <state_interface name="velocity"/>
+        </joint>
+    </ros2_control>
+</robot>
+<!--
 <?xml version="1.0"?>
 <robot xmlns:xacro="http://www.ros.org/wiki/xacro">
@@ -27,23 +48,3 @@
         </plugin>
     </gazebo>
-</robot>
-<!-- <?xml version="1.0"?>
-<robot xmlns:xacro="http://www.ros.org/wiki/xacro">
-    <ros2_control name="RealRobot" type="system">
-        <hardware>
-            <plugin>hinson_hardware/HinsonSystemHardware</plugin>
-            <param name="port">/dev/ttyUSB0</param>
-            <param name="baudrate">115200</param>
-        </hardware>
-        <joint name="left_wheel_joint">
-            <command_interface name="velocity"/>
-            <state_interface name="position"/>
-            <state_interface name="velocity"/>
-        </joint>
-        <joint name="right_wheel_joint">
-            <command_interface name="velocity"/>
-            <state_interface name="position"/>
-            <state_interface name="velocity"/>
-        </joint>
-    </ros2_control>
 </robot> -->

Commit message: feat: tích hợp Nav2, IMU driver, web bridge và dọn workspace, web cơ bản dùng chung wifi

File: src/amr_lan_3/description/robot_core.xacro (robot description, xacro)
@@ -289,3 +289,48 @@
         <slip2>1.0</slip2> -->
     </gazebo>
+    <joint name="imu_joint" type="fixed">
+        <parent link="base_link"/>
+        <child link="imu_link"/>
+        <origin xyz="0.0 0.0 0.05" rpy="0 0 0"/>
+    </joint>
+    <link name="imu_link">
+        <visual>
+            <origin xyz="0 0 0"/>
+            <geometry>
+                <box size="0.03 0.03 0.01"/>
+            </geometry>
+            <material name="black"/>
+        </visual>
+        <collisopn>
+            <origin xyz="0 0 0"/>
+            <geometry>
+                <box size="0.03 0.03 0.01"/>
+            </geometry>
+        </collisopn>
+        <xacro:inertial_box mass="0.01" x="0.03" y="0.03" z="0.01">
+            <origin xyz="0 0 0" rpy="0 0 0"/>
+        </xacro:inertial_box>
+    </link>
+    <gazebo reference="imu_link">
+        <gravity>true</gravity>
+        <sensor name="imu_sensor" type="imu">
+            <always_on>true</always_on>
+            <update_rate>100</update_rate> <visualize>true</visualize>
+            <topic>/imu/data</topic>
+            <plugin filename="libgazebo_ros_imu_sensor.so" name="imu_plugin">
+                <ros>
+                    <remapping>~/out:=/imu/data</remapping>
+                </ros>
+                <!-- <topicName>/imu/data</topicName> -->
+                <bodyName>imu_link</bodyName>
+                <updateRateHZ>100.0</updateRateHZ>
+                <gaussianNoise>0.002</gaussianNoise> <xyzOffset>0 0 0</xyzOffset>
+                <rpyOffset>0 0 0</rpyOffset>
+                <frameName>imu_link</frameName>
+                <initialOrientationAsReference>false</initialOrientationAsReference>
+            </plugin>
+            <pose>0 0 0 0 0 0</pose>
+        </sensor>
+        <material>Gazebo/Black</material>
+    </gazebo>
 </robot>
