Commit message: feat: tich hop driver rplidar vao nhanh slam
Quet ban do bang SLAM toolbox su dung odom va Lidar A1M8, ca mo phong va real robot

File: src/amr_lan_3/description/gazebo_control.xacro (robot description, xacro)
@@ -7,5 +7,8 @@
             <right_joint>right_wheel_joint</right_joint>
              <!-- o origin trong tag joint -->
-            <wheel_separation>0.56</wheel_separation>
+            <!-- <wheel_separation>0.56</wheel_separation> -->
+            <!-- <wheel_separation>0.594</wheel_separation>  -->
+            <!-- <wheel_separation>0.553</wheel_separation>  -->
+            <wheel_separation>0.568</wheel_separation>
             <wheel_diameter>0.18</wheel_diameter>
             <!-- Limits -->

File: src/amr_lan_3/description/robot_core.xacro (robot description, xacro)
@@ -72,5 +72,7 @@
             <origin xyz="0 0 0"/>
             <geometry>
-                <box size="1.04 0.51 0.06"/>
+                <!-- <box size="1.04 0.51 0.06"/> -->
+                <!-- <box size="1.05 0.54 0.06"/> -->
+                <box size="1.1 0.6 0.06"/>
             </geometry>
             <material name="vibrantorange"/>
@@ -79,5 +81,7 @@
             <origin xyz="0 0 0"/>
             <geometry>
-                <box size="1.04 0.51 0.06"/>
+                <!-- <box size="1.04 0.51 0.06"/> -->
+                <!-- <box size="1.05 0.54 0.06"/> -->
+                <box size="1.1 0.6 0.06"/>
             </geometry>
         </collision>
@@ -93,5 +97,9 @@
         <parent link="base_link"/>
         <child link="left_wheel"/>
-        <origin xyz="0 0.28 0" rpy="-${pi/2} 0 0"/>
+        <!-- <origin xyz="0 0.28 0" rpy="-${pi/2} 0 0"/> -->
+        <!-- <origin xyz="0 0.297 0" rpy="-${pi/2} 0 0"/> -->
+        <!-- <origin xyz="0 0.288 0" rpy="-${pi/2} 0 0"/> -->
+        <!-- <origin xyz="0 0.2765 0" rpy="-${pi/2} 0 0"/> -->
+         <origin xyz="0 0.284 0" rpy="-${pi/2} 0 0"/>
         <axis xyz="0 0 1"/>
     </joint>
@@ -100,5 +108,6 @@
             <origin xyz="0 0 0"/>
             <geometry>
-                <cylinder radius="0.09" length="0.04"/>
+                <!-- <cylinder radius="0.09" length="0.04"/> -->
+                <cylinder radius="0.09" length="0.046"/>
             </geometry>
             <material name="tim"/>
@@ -111,5 +120,5 @@
             </geometry>
         </collision>
-        <xacro:inertial_cylinder mass = "1.5" length="0.04" radius="0.09">
+        <xacro:inertial_cylinder mass = "1.5" length="0.046" radius="0.09">
             <origin xyz="0 0 0" rpy="0 0 0"/>
         </xacro:inertial_cylinder>
@@ -124,5 +133,9 @@
         <parent link="base_link"/>
         <child link="right_wheel"/>
-        <origin xyz="0 -0.28 0" rpy="${pi/2} 0 0"/>
+        <!-- <origin xyz="0 -0.28 0" rpy="${pi/2} 0 0"/> -->
+        <!-- <origin xyz="0 -0.297 0" rpy="${pi/2} 0 0"/> -->
+        <!-- <origin xyz="0 -0.288 0" rpy="${pi/2} 0 0"/> -->
+        <!-- <origin xyz="0 -0.2765 0" rpy="${pi/2} 0 0"/> -->
+        <origin xyz="0 -0.284 0" rpy="${pi/2} 0 0"/>
         <axis xyz="0 0 -1"/>
     </joint>
@@ -131,5 +144,6 @@
             <origin xyz="0 0 0"/>
             <geometry>
-                <cylinder radius="0.09" length="0.04"/>
+                <!-- <cylinder radius="0.09" length="0.04"/> -->
+                <cylinder radius="0.09" length="0.046"/>
             </geometry>
             <material name="tim"/>
@@ -142,5 +156,5 @@
             </geometry>
         </collision>
-        <xacro:inertial_cylinder mass = "1.5" length="0.04" radius="0.09">
+        <xacro:inertial_cylinder mass = "1.5" length="0.046" radius="0.09">
             <origin xyz="0 0 0" rpy="0 0 0"/>
         </xacro:inertial_cylinder>

File: src/amr_lan_3/description/ros2_control.xacro (robot description, xacro)
@@ -5,5 +5,6 @@
             <hardware>
                 <plugin>hinson_hardware/HinsonSystemHardware</plugin>
-                <param name="port">/dev/ttyUSB0</param>
+                <param name="port">/dev/serial/by-id/usb-FTDI_FT232R_USB_UART_A5069RR4-if00-port0</param>
+                <!-- <param name="port">/dev/ttyUSB0</param> -->
                 <param name="baudrate">115200</param>
             </hardware>

Commit message: Update slam, nav2 params

File: src/amr_lan_3/description/gazebo_control.xacro (robot description, xacro)
@@ -10,5 +10,6 @@
             <!-- <wheel_separation>0.594</wheel_separation>  -->
             <!-- <wheel_separation>0.553</wheel_separation>  -->
-            <wheel_separation>0.568</wheel_separation>
+            <!-- <wheel_separation>0.568</wheel_separation> bua  -->
+            <wheel_separation>0.572</wheel_separation>
             <wheel_diameter>0.18</wheel_diameter>
             <!-- Limits -->

File: src/amr_lan_3/description/robot_core.xacro (robot description, xacro)
@@ -101,5 +101,8 @@
         <!-- <origin xyz="0 0.288 0" rpy="-${pi/2} 0 0"/> -->
         <!-- <origin xyz="0 0.2765 0" rpy="-${pi/2} 0 0"/> -->
-         <origin xyz="0 0.284 0" rpy="-${pi/2} 0 0"/>
+         <!-- <origin xyz="0 0.284 0" rpy="-${pi/2} 0 0"/> bua  -->
+         <!-- <origin xyz="0 0.286 0" rpy="-${pi/2} 0 0"/> 24_06_2026 -->
+         <!-- 26_06_2026 -->
+        <origin xyz="0 0.28515 0" rpy="-${pi/2} 0 0"/>
         <axis xyz="0 0 1"/>
     </joint>
@@ -137,5 +140,8 @@
         <!-- <origin xyz="0 -0.288 0" rpy="${pi/2} 0 0"/> -->
         <!-- <origin xyz="0 -0.2765 0" rpy="${pi/2} 0 0"/> -->
-        <origin xyz="0 -0.284 0" rpy="${pi/2} 0 0"/>
+        <!-- <origin xyz="0 -0.284 0" rpy="${pi/2} 0 0"/> bua  -->
+        <!-- <origin xyz="0 -0.286 0" rpy="${pi/2} 0 0"/> 24_06_2026 -->
+        <!-- 26_06_2026 -->
+        <origin xyz="0 -0.28515 0" rpy="${pi/2} 0 0"/>
         <axis xyz="0 0 -1"/>
     </joint>
